Commit message: Add better worlds

File: coug_gazebo/worlds/byu.sdf.xacro (robot description, xacro)
@@ -15,6 +15,6 @@
   <xacro:arg name="headless" default="true" />
   <xacro:property name="terrain_dir" value="$(find coug_gazebo)/models/byu_terrain" />
-  <xacro:property name="terrain_size" value="1129.9 1629.95 63.61" />
-  <xacro:property name="terrain_z" value="-30.72" />
+  <xacro:property name="terrain_size" value="1129.9 1629.95 63.67" />
+  <xacro:property name="terrain_z" value="-30.74" />
   <world name="default">
     <plugin filename="gz-sim-physics-system" name="gz::sim::systems::Physics" />
@@ -37,5 +37,5 @@
       <latitude_deg>40.2515095</latitude_deg>
       <longitude_deg>-111.6496175</longitude_deg>
-      <elevation>1424.159</elevation>
+      <elevation>1424.162</elevation>
     </spherical_coordinates>
     <light type="directional" name="sun">

File: coug_gazebo/worlds/mdrs.sdf.xacro (robot description, xacro)
@@ -15,6 +15,8 @@
   <xacro:arg name="headless" default="true" />
   <xacro:property name="terrain_dir" value="$(find coug_gazebo)/models/mdrs_terrain" />
-  <xacro:property name="terrain_size" value="2005.08 1996.57 71.3" />
+  <xacro:property name="terrain_size" value="2005.08 1996.57 71.36" />
   <xacro:property name="terrain_z" value="-13.67" />
+  <xacro:property name="aruco_mesh" value="$(find coug_gazebo)/models/urc_aruco_1/meshes/urc_aruco_1.dae" />
+  <xacro:property name="aruco_texture" value="$(find coug_gazebo)/models/urc_aruco_1/meshes/urc_aruco_1.png" />
   <world name="default">
     <plugin filename="gz-sim-physics-system" name="gz::sim::systems::Physics" />
@@ -37,5 +39,5 @@
       <latitude_deg>38.406</latitude_deg>
       <longitude_deg>-110.792</longitude_deg>
-      <elevation>1373.134</elevation>
+      <elevation>1373.153</elevation>
     </spherical_coordinates>
     <light type="directional" name="sun">
@@ -82,4 +84,45 @@
       </link>
     </model>
+    <!-- ArUco tag 1 (4X4_50) on a post, beside the rover spawn -->
+    <model name="aruco_1">
+      <static>true</static>
+      <pose>-9 -13 -0.2 0 0 0</pose>
+      <link name="link">
+        <collision name="tag_collision">
+          <geometry>
+            <mesh>
+              <uri>${aruco_mesh}</uri>
+            </mesh>
+          </geometry>
+        </collision>
+        <visual name="tag_visual">
+          <geometry>
+            <mesh>
+              <uri>${aruco_mesh}</uri>
+            </mesh>
+          </geometry>
+          <material>
+            <ambient>1 1 1 1</ambient>
+            <diffuse>1 1 1 1</diffuse>
+            <pbr>
+              <metal>
+                <albedo_map>${aruco_texture}</albedo_map>
+                <roughness>1.0</roughness>
+                <metalness>0.0</metalness>
+              </metal>
+            </pbr>
+          </material>
+        </visual>
+        <visual name="post_visual">
+          <pose>0 0 -1.5 0 0 0</pose>
+          <geometry>
+            <cylinder>
+              <radius>0.02</radius>
+              <length>3.0</length>
+            </cylinder>
+          </geometry>
+        </visual>
+      </link>
+    </model>
   </world>
 </sdf>

Commit message: Add default mock

File: coug_gazebo/worlds/byu.sdf.xacro (robot description, xacro)
@@ -17,4 +17,5 @@
   <xacro:property name="terrain_size" value="1129.9 1629.95 63.67" />
   <xacro:property name="terrain_z" value="-30.74" />
+  <xacro:include filename="aruco_tag.xacro" />
   <world name="default">
     <plugin filename="gz-sim-physics-system" name="gz::sim::systems::Physics" />

File: coug_gazebo/worlds/mdrs.sdf.xacro (robot description, xacro)
@@ -17,6 +17,5 @@
   <xacro:property name="terrain_size" value="2005.08 1996.57 71.36" />
   <xacro:property name="terrain_z" value="-13.67" />
-  <xacro:property name="aruco_mesh" value="$(find coug_gazebo)/models/urc_aruco_1/meshes/urc_aruco_1.dae" />
-  <xacro:property name="aruco_texture" value="$(find coug_gazebo)/models/urc_aruco_1/meshes/urc_aruco_1.png" />
+  <xacro:include filename="aruco_tag.xacro" />
   <world name="default">
     <plugin filename="gz-sim-physics-system" name="gz::sim::systems::Physics" />
@@ -84,45 +83,7 @@
       </link>
     </model>
-    <!-- ArUco tag 1 (4X4_50) on a post, beside the rover spawn -->
-    <model name="aruco_1">
-      <static>true</static>
-      <pose>-9 -13 -0.2 0 0 0</pose>
-      <link name="link">
-        <collision name="tag_collision">
-          <geometry>
-            <mesh>
-              <uri>${aruco_mesh}</uri>
-            </mesh>
-          </geometry>
-        </collision>
-        <visual name="tag_visual">
-          <geometry>
-            <mesh>
-              <uri>${aruco_mesh}</uri>
-            </mesh>
-          </geometry>
-          <material>
-            <ambient>1 1 1 1</ambient>
-            <diffuse>1 1 1 1</diffuse>
-            <pbr>
-              <metal>
-                <albedo_map>${aruco_texture}</albedo_map>
-                <roughness>1.0</roughness>
-                <metalness>0.0</metalness>
-              </metal>
-            </pbr>
-          </material>
-        </visual>
-        <visual name="post_visual">
-          <pose>0 0 -1.5 0 0 0</pose>
-          <geometry>
-            <cylinder>
-              <radius>0.02</radius>
-              <length>3.0</length>
-            </cylinder>
-          </geometry>
-        </visual>
-      </link>
-    </model>
+    <xacro:aruco_tag id="0" pose="-5 -7 -0.86 0 0 0" />
+    <xacro:aruco_tag id="1" pose="20 27 -0.58 0 0 0" />
+    <xacro:aruco_tag id="2" pose="-72 72 7.54 0 0 0" />
   </world>
 </sdf>

File: coug_gazebo/worlds/sonoma_raceway.sdf.xacro (robot description, xacro)
@@ -14,4 +14,5 @@
 <sdf version="1.9" xmlns:xacro="http://www.ros.org/wiki/xacro">
   <xacro:arg name="headless" default="true" />
+  <xacro:include filename="aruco_tag.xacro" />
   <world name="default">
     <plugin filename="gz-sim-physics-system" name="gz::sim::systems::Physics" />

File: coug_gazebo/worlds/urc.sdf.xacro (robot description, xacro)
@@ -17,4 +17,5 @@
   <xacro:property name="terrain_size" value="2000.0 2000.0 85.71" />
   <xacro:property name="terrain_z" value="-48.88" />
+  <xacro:include filename="aruco_tag.xacro" />
   <world name="default">
     <plugin filename="gz-sim-physics-system" name="gz::sim::systems::Physics" />

Commit message: Better world organization

File: coug_gazebo/worlds/byu.sdf.xacro (robot description, xacro)
@@ -14,73 +14,20 @@
 <sdf version="1.9" xmlns:xacro="http://www.ros.org/wiki/xacro">
   <xacro:arg name="headless" default="true" />
+  <xacro:include filename="world_common.xacro" />
   <xacro:property name="terrain_dir" value="$(find coug_gazebo)/models/byu_terrain" />
-  <xacro:property name="terrain_size" value="1129.9 1629.95 63.67" />
-  <xacro:property name="terrain_z" value="-30.74" />
-  <xacro:include filename="aruco_tag.xacro" />
   <world name="default">
-    <plugin filename="gz-sim-physics-system" name="gz::sim::systems::Physics" />
-    <plugin filename="gz-sim-user-commands-system" name="gz::sim::systems::UserCommands" />
-    <plugin filename="gz-sim-navsat-system" name="gz::sim::systems::NavSat" />
-    <xacro:unless value="$(arg headless)">
-      <plugin filename="gz-sim-scene-broadcaster-system" name="gz::sim::systems::SceneBroadcaster" />
-    </xacro:unless>
-    <plugin filename="gz-sim-sensors-system" name="gz::sim::systems::Sensors">
-      <render_engine>ogre2</render_engine>
-    </plugin>
-    <plugin filename="gz-sim-imu-system" name="gz::sim::systems::Imu" />
-    <plugin filename="gz-sim-magnetometer-system" name="gz::sim::systems::Magnetometer">
-      <use_units_gauss>false</use_units_gauss>
-      <use_earth_frame_ned>false</use_earth_frame_ned>
-    </plugin>
-    <spherical_coordinates>
-      <surface_model>EARTH_WGS84</surface_model>
-      <world_frame_orientation>ENU</world_frame_orientation>
-      <latitude_deg>40.2515095</latitude_deg>
-      <longitude_deg>-111.6496175</longitude_deg>
-      <elevation>1424.162</elevation>
-    </spherical_coordinates>
-    <light type="directional" name="sun">
-      <cast_shadows>true</cast_shadows>
-      <specular>0 0 0 1</specular>
-      <direction>0 0.6 -0.6</direction>
-    </light>
+    <xacro:world_systems headless="$(arg headless)" />
+    <xacro:world_origin latitude="40.2515095" longitude="-111.6496175" elevation="1424.162" />
+    <xacro:sun />
     <scene>
       <sky />
     </scene>
-    <!-- Heightmaps need the bullet collision detector -->
-    <physics type="dart">
-      <max_step_size>0.003</max_step_size>
-      <dart>
-        <collision_detector>bullet</collision_detector>
-      </dart>
-    </physics>
-    <model name="byu_terrain">
-      <static>true</static>
-      <link name="ground">
-        <collision name="collision">
-          <pose>0 0 ${terrain_z} 0 0 0</pose>
-          <geometry>
-            <heightmap>
-              <uri>${terrain_dir}/height_map.png</uri>
-              <size>${terrain_size}</size>
-            </heightmap>
-          </geometry>
-        </collision>
-        <visual name="visual">
-          <geometry>
-            <heightmap>
-              <uri>${terrain_dir}/height_map.png</uri>
-              <size>${terrain_size}</size>
-              <pos>0 0 ${terrain_z}</pos>
-              <texture>
-                <diffuse>${terrain_dir}/aerial.png</diffuse>
-                <normal>${terrain_dir}/normal_map.png</normal>
-                <size>1629.95</size>
-              </texture>
-            </heightmap>
-          </geometry>
-        </visual>
-      </link>
-    </model>
+    <xacro:heightmap_physics />
+    <xacro:heightmap_terrain
+      name="byu_terrain"
+      dir="${terrain_dir}"
+      size="1129.9 1629.95 63.67"
+      z="-30.74"
+    />
     <model name="byu_buildings">
       <static>true</static>

File: coug_gazebo/worlds/mdrs.sdf.xacro (robot description, xacro)
@@ -14,73 +14,19 @@
 <sdf version="1.9" xmlns:xacro="http://www.ros.org/wiki/xacro">
   <xacro:arg name="headless" default="true" />
-  <xacro:property name="terrain_dir" value="$(find coug_gazebo)/models/mdrs_terrain" />
-  <xacro:property name="terrain_size" value="2005.08 1996.57 71.36" />
-  <xacro:property name="terrain_z" value="-13.67" />
-  <xacro:include filename="aruco_tag.xacro" />
+  <xacro:include filename="world_common.xacro" />
   <world name="default">
-    <plugin filename="gz-sim-physics-system" name="gz::sim::systems::Physics" />
-    <plugin filename="gz-sim-user-commands-system" name="gz::sim::systems::UserCommands" />
-    <plugin filename="gz-sim-navsat-system" name="gz::sim::systems::NavSat" />
-    <xacro:unless value="$(arg headless)">
-      <plugin filename="gz-sim-scene-broadcaster-system" name="gz::sim::systems::SceneBroadcaster" />
-    </xacro:unless>
-    <plugin filename="gz-sim-sensors-system" name="gz::sim::systems::Sensors">
-      <render_engine>ogre2</render_engine>
-    </plugin>
-    <plugin filename="gz-sim-imu-system" name="gz::sim::systems::Imu" />
-    <plugin filename="gz-sim-magnetometer-system" name="gz::sim::systems::Magnetometer">
-      <use_units_gauss>false</use_units_gauss>
-      <use_earth_frame_ned>false</use_earth_frame_ned>
-    </plugin>
-    <spherical_coordinates>
-      <surface_model>EARTH_WGS84</surface_model>
-      <world_frame_orientation>ENU</world_frame_orientation>
-      <latitude_deg>38.406</latitude_deg>
-      <longitude_deg>-110.792</longitude_deg>
-      <elevation>1373.153</elevation>
-    </spherical_coordinates>
-    <light type="directional" name="sun">
-      <cast_shadows>true</cast_shadows>
-      <specular>0 0 0 1</specular>
-      <direction>0 0.6 -0.6</direction>
-    </light>
+    <xacro:world_systems headless="$(arg headless)" />
+    <xacro:world_origin latitude="38.406" longitude="-110.792" elevation="1373.153" />
+    <xacro:sun />
     <scene>
       <sky />
     </scene>
-    <!-- Heightmaps need the bullet collision detector -->
-    <physics type="dart">
-      <max_step_size>0.003</max_step_size>
-      <dart>
-        <collision_detector>bullet</collision_detector>
-      </dart>
-    </physics>
-    <model name="mdrs_terrain">
-      <static>true</static>
-      <link name="ground">
-        <collision name="collision">
-          <pose>0 0 ${terrain_z} 0 0 0</pose>
-          <geometry>
-            <heightmap>
-              <uri>${terrain_dir}/height_map.png</uri>
-              <size>${terrain_size}</size>
-            </heightmap>
-          </geometry>
-        </collision>
-        <visual name="visual">
-          <geometry>
-            <heightmap>
-              <uri>${terrain_dir}/height_map.png</uri>
-              <size>${terrain_size}</size>
-              <pos>0 0 ${terrain_z}</pos>
-              <texture>
-                <diffuse>${terrain_dir}/aerial.png</diffuse>
-                <normal>${terrain_dir}/normal_map.png</normal>
-                <size>2005.08</size>
-              </texture>
-            </heightmap>
-          </geometry>
-        </visual>
-      </link>
-    </model>
+    <xacro:heightmap_physics />
+    <xacro:heightmap_terrain
+      name="mdrs_terrain"
+      dir="$(find coug_gazebo)/models/mdrs_terrain"
+      size="2005.08 1996.57 71.36"
+      z="-13.67"
+    />
     <xacro:aruco_tag id="0" pose="-5 -7 -0.86 0 0 0" />
     <xacro:aruco_tag id="1" pose="20 27 -0.58 0 0 0" />

File: coug_gazebo/worlds/sonoma_raceway.sdf.xacro (robot description, xacro)
@@ -14,31 +14,9 @@
 <sdf version="1.9" xmlns:xacro="http://www.ros.org/wiki/xacro">
   <xacro:arg name="headless" default="true" />
-  <xacro:include filename="aruco_tag.xacro" />
+  <xacro:include filename="world_common.xacro" />
   <world name="default">
-    <plugin filename="gz-sim-physics-system" name="gz::sim::systems::Physics" />
-    <plugin filename="gz-sim-user-commands-system" name="gz::sim::systems::UserCommands" />
-    <plugin filename="gz-sim-navsat-system" name="gz::sim::systems::NavSat" />
-    <xacro:unless value="$(arg headless)">
-      <plugin filename="gz-sim-scene-broadcaster-system" name="gz::sim::systems::SceneBroadcaster" />
-    </xacro:unless>
-    <plugin filename="gz-sim-sensors-system" name="gz::sim::systems::Sensors">
-      <render_engine>ogre2</render_engine>
-    </plugin>
-    <plugin filename="gz-sim-imu-system" name="gz::sim::systems::Imu" />
-    <plugin filename="gz-sim-magnetometer-system" name="gz::sim::systems::Magnetometer">
-      <use_units_gauss>false</use_units_gauss>
-      <use_earth_frame_ned>false</use_earth_frame_ned>
-    </plugin>
-    <spherical_coordinates>
-      <surface_model>EARTH_WGS84</surface_model>
-      <world_frame_orientation>ENU</world_frame_orientation>
-      <latitude_deg>38.161479</latitude_deg>
-      <longitude_deg>-122.454630</longitude_deg>
-      <elevation>6.39</elevation>
-    </spherical_coordinates>
-    <light type="directional" name="sun">
-      <cast_shadows>true</cast_shadows>
-      <direction>0 0.6 -0.6</direction>
-    </light>
+    <xacro:world_systems headless="$(arg headless)" />
+    <xacro:world_origin latitude="38.161479" longitude="-122.454630" elevation="6.39" />
+    <xacro:sun />
     <scene>
       <sky />

File: coug_gazebo/worlds/urc.sdf.xacro (robot description, xacro)
@@ -14,73 +14,19 @@
 <sdf version="1.9" xmlns:xacro="http://www.ros.org/wiki/xacro">
   <xacro:arg name="headless" default="true" />
-  <xacro:property name="terrain_dir" value="$(find coug_gazebo)/models/urc_terrain" />
-  <xacro:property name="terrain_size" value="2000.0 2000.0 85.71" />
-  <xacro:property name="terrain_z" value="-48.88" />
-  <xacro:include filename="aruco_tag.xacro" />
+  <xacro:include filename="world_common.xacro" />
   <world name="default">
-    <plugin filename="gz-sim-physics-system" name="gz::sim::systems::Physics" />
-    <plugin filename="gz-sim-user-commands-system" name="gz::sim::systems::UserCommands" />
-    <plugin filename="gz-sim-navsat-system" name="gz::sim::systems::NavSat" />
-    <xacro:unless value="$(arg headless)">
-      <plugin filename="gz-sim-scene-broadcaster-system" name="gz::sim::systems::SceneBroadcaster" />
-    </xacro:unless>
-    <plugin filename="gz-sim-sensors-system" name="gz::sim::systems::Sensors">
-      <render_engine>ogre2</render_engine>
-    </plugin>
-    <plugin filename="gz-sim-imu-system" name="gz::sim::systems::Imu" />
-    <plugin filename="gz-sim-magnetometer-system" name="gz::sim::systems::Magnetometer">
-      <use_units_gauss>false</use_units_gauss>
-      <use_earth_frame_ned>false</use_earth_frame_ned>
-    </plugin>
-    <spherical_coordinates>
-      <surface_model>EARTH_WGS84</surface_model>
-      <world_frame_orientation>ENU</world_frame_orientation>
-      <latitude_deg>38.418</latitude_deg>
-      <longitude_deg>-110.777</longitude_deg>
-      <elevation>1394.024</elevation>
-    </spherical_coordinates>
-    <light type="directional" name="sun">
-      <cast_shadows>true</cast_shadows>
-      <specular>0 0 0 1</specular>
-      <direction>0 0.6 -0.6</direction>
-    </light>
+    <xacro:world_systems headless="$(arg headless)" />
+    <xacro:world_origin latitude="38.418" longitude="-110.777" elevation="1394.024" />
+    <xacro:sun />
     <scene>
       <sky />
     </scene>
-    <!-- Heightmaps need the bullet collision detector -->
-    <physics type="dart">
-      <max_step_size>0.003</max_step_size>
-      <dart>
-        <collision_detector>bullet</collision_detector>
-      </dart>
-    </physics>
-    <model name="urc_terrain">
-      <static>true</static>
-      <link name="ground">
-        <collision name="collision">
-          <pose>0 0 ${terrain_z} 0 0 0</pose>
-          <geometry>
-            <heightmap>
-              <uri>${terrain_dir}/height_map.png</uri>
-              <size>${terrain_size}</size>
-            </heightmap>
-          </geometry>
-        </collision>
-        <visual name="visual">
-          <geometry>
-            <heightmap>
-              <uri>${terrain_dir}/height_map.png</uri>
-              <size>${terrain_size}</size>
-              <pos>0 0 ${terrain_z}</pos>
-              <texture>
-                <diffuse>${terrain_dir}/aerial.png</diffuse>
-                <normal>${terrain_dir}/normal_map.png</normal>
-                <size>2000.0</size>
-              </texture>
-            </heightmap>
-          </geometry>
-        </visual>
-      </link>
-    </model>
+    <xacro:heightmap_physics />
+    <xacro:heightmap_terrain
+      name="urc_terrain"
+      dir="$(find coug_gazebo)/models/urc_terrain"
+      size="2000.0 2000.0 85.71"
+      z="-48.88"
+    />
   </world>
 </sdf>

Commit message: Better aruco models

File: coug_gazebo/worlds/byu.sdf.xacro (robot description, xacro)
@@ -48,10 +48,10 @@
       </link>
     </model>
-    <xacro:aruco_tag id="0" pose="74 -553 -5.09 0 0 0" />
-    <xacro:aruco_tag id="1" pose="54 -572 -4.93 0 0 0" />
-    <xacro:aruco_tag id="2" pose="45 -555 -4.39 0 0 0" />
-    <xacro:aruco_tag id="3" pose="50 -593 -5.92 0 0 0" />
-    <xacro:aruco_tag id="4" pose="20 -560 -4.59 0 0 0" />
-    <xacro:aruco_tag id="5" pose="16 -594 -5.88 0 0 0" />
+    <xacro:urc_aruco_w_post id="0" pose="74 -553 -5.09 0 0 0" />
+    <xacro:urc_aruco_w_post id="1" pose="54 -572 -4.93 0 0 0" />
+    <xacro:urc_aruco_w_post id="2" pose="45 -555 -4.39 0 0 0" />
+    <xacro:urc_aruco_w_post id="3" pose="50 -593 -5.92 0 0 0" />
+    <xacro:urc_aruco_w_post id="4" pose="20 -560 -4.59 0 0 0" />
+    <xacro:urc_aruco_w_post id="5" pose="16 -594 -5.88 0 0 0" />
   </world>
 </sdf>

File: coug_gazebo/worlds/mdrs.sdf.xacro (robot description, xacro)
@@ -24,7 +24,7 @@
     <xacro:heightmap_physics />
     <xacro:heightmap_terrain name="mdrs_terrain" dir="$(find coug_gazebo)/models/mdrs_terrain" size="2005.08 1996.57 71.36" z="-13.67" />
-    <xacro:aruco_tag id="0" pose="-5 -7 -0.86 0 0 0" />
-    <xacro:aruco_tag id="1" pose="20 27 -0.58 0 0 0" />
-    <xacro:aruco_tag id="2" pose="-72 72 7.54 0 0 0" />
+    <xacro:urc_aruco_w_post id="0" pose="-5 -7 -0.86 0 0 0" />
+    <xacro:urc_aruco_w_post id="1" pose="20 27 -0.58 0 0 0" />
+    <xacro:urc_aruco_w_post id="2" pose="-72 72 7.54 0 0 0" />
   </world>
 </sdf>

File: coug_gazebo/worlds/world_common.xacro (robot description, xacro)
@@ -83,28 +83,10 @@
     </model>
   </xacro:macro>
-  <xacro:macro name="aruco_tag" params="id pose height:=1.0">
-    <model name="aruco_${id}">
-      <static>true</static>
+  <xacro:macro name="urc_aruco_w_post" params="id pose">
+    <include>
+      <uri>model://urc_aruco_${id}_w_post</uri>
+      <name>aruco_${id}</name>
       <pose>${pose}</pose>
-      <link name="link">
-        <visual name="tag_visual">
-          <pose>0 0 ${height} 0 0 0</pose>
-          <geometry>
-            <mesh>
-              <uri>$(find coug_gazebo)/models/urc_aruco_${id}/urc_aruco_${id}.dae</uri>
-            </mesh>
-          </geometry>
-        </visual>
-        <visual name="post_visual">
-          <pose>0 0 ${(height - 0.5) / 2} 0 0 0</pose>
-          <geometry>
-            <cylinder>
-              <radius>0.02</radius>
-              <length>${height + 0.5}</length>
-            </cylinder>
-          </geometry>
-        </visual>
-      </link>
-    </model>
+    </include>
   </xacro:macro>
 </sdf>
