Commit message: Lidar working on blueboat

File: coug_gazebo/urdf/blueboat.gazebo.xacro (robot description, xacro)
@@ -119,7 +119,8 @@
     </sensor>
   </gazebo>
-  <xacro:imu_sensors link="${tf_prefix}depth_camera_link" />
+  <xacro:imu_sensors link="${tf_prefix}imu_link" />
   <xacro:gps_sensor link="${tf_prefix}gps_link" />
-  <xacro:depth_camera_sensor link="${tf_prefix}depth_camera_link" />
+  <xacro:lidar_sensor link="${tf_prefix}lidar_link" />
+  <xacro:rgb_camera_sensor link="${tf_prefix}depth_camera_link" />
   <xacro:boundingbox_camera_sensor link="${tf_prefix}depth_camera_link" />
 </robot>

File: coug_gazebo/urdf/sensors.gazebo.xacro (robot description, xacro)
@@ -118,5 +118,5 @@
     </gazebo>
   </xacro:macro>
-  <xacro:macro name="depth_camera_sensor" params="link">
+  <xacro:macro name="rgb_camera_sensor" params="link">
     <gazebo reference="${link}">
       <sensor name="rgb_camera" type="camera">
@@ -144,4 +144,9 @@
         </camera>
       </sensor>
+    </gazebo>
+  </xacro:macro>
+  <xacro:macro name="depth_camera_sensor" params="link">
+    <xacro:rgb_camera_sensor link="${link}" />
+    <gazebo reference="${link}">
       <sensor name="depth_camera" type="rgbd_camera">
         <always_on>true</always_on>
@@ -204,3 +209,38 @@
     </gazebo>
   </xacro:macro>
+  <xacro:macro name="lidar_sensor" params="link">
+    <gazebo reference="${link}">
+      <sensor name="lidar" type="gpu_lidar">
+        <always_on>true</always_on>
+        <!-- https://data.ouster.io/downloads/datasheets/datasheet-rev7-v3p1-os1.pdf -->
+        <update_rate>10</update_rate>
+        <topic>/${agent_ns}/lidar</topic>
+        <gz_frame_id>${link}</gz_frame_id>
+        <lidar>
+          <!-- https://data.ouster.io/downloads/datasheets/datasheet-rev7-v3p1-os1.pdf -->
+          <scan>
+            <horizontal>
+              <samples>1024</samples>
+              <min_angle>${-pi}</min_angle>
+              <max_angle>${pi}</max_angle>
+            </horizontal>
+            <vertical>
+              <samples>64</samples>
+              <min_angle>${radians(-21.2)}</min_angle>
+              <max_angle>${radians(21.2)}</max_angle>
+            </vertical>
+          </scan>
+          <!-- https://data.ouster.io/downloads/datasheets/datasheet-rev7-v3p1-os1.pdf -->
+          <range>
+            <min>0.5</min>
+            <max>90.0</max>
+          </range>
+          <noise type="gaussian">
+            <mean>0.0</mean>
+            <stddev>0.01</stddev>
+          </noise>
+        </lidar>
+      </sensor>
+    </gazebo>
+  </xacro:macro>
 </robot>
